File: electronics/boards/starter/rev-a/inputs.kicad_sch (KiCad schematic)
At the start: 19 parts, among them J10 3-POSITION SELECTOR, J5 10k LINEAR AXIS POT, J7 HAT N E S W, J8 ENCODER A B PUSH, J9 MAINTAINED TOGGLE

Commit message: Review compact four-layer PCB and add milling qualification coupon
Parts:
- C12: MPN (none) -> C0805C104K3RACTU
- J10, J5: footprint KiCad:PinHeader_1x03_P2.54mm_Vertical -> OpenSimGear:PinHeader_Samtec_TSW-103-07-L-S_P2.54mm_Vertical; MPN (none) -> TSW-103-07-L-S
- J7: footprint KiCad:PinHeader_1x05_P2.54mm_Vertical -> OpenSimGear:PinHeader_Samtec_TSW-105-07-L-S_P2.54mm_Vertical; MPN (none) -> TSW-105-07-L-S
- J8: footprint KiCad:PinHeader_1x04_P2.54mm_Vertical -> OpenSimGear:PinHeader_Samtec_TSW-104-07-L-S_P2.54mm_Vertical; MPN (none) -> TSW-104-07-L-S
- J9: footprint KiCad:PinHeader_1x02_P2.54mm_Vertical -> OpenSimGear:PinHeader_Samtec_TSW-102-07-L-S_P2.54mm_Vertical; MPN (none) -> TSW-102-07-L-S
- R10, R11, R12, R13, R14, R15, R16, R17, R18, R9: MPN (none) -> RC0805FR-0710KL
- R19: MPN (none) -> RC0805FR-071KL
- R20, R21: MPN (none) -> RC0805FR-071ML
