File: electronics/boards/starter/rev-a/starter.kicad_sch (KiCad schematic)
At the start: 41 parts, among them J1 USB-C DEVICE, J2 12V CAN - NOT PHONE, J3 12V CAN - NOT PHONE, J4 SWD / 3V3 REFERENCE ONLY, J5 GPIO 3V3, J6 CAN TEST / END TERMINATION, SW1 TEST BUTTON, SW2 RESET, U1 STM32G0B1CBT6, U2 USBLC6-2SC6, U3 TCAN3413D, U4 R-78E5.0-0.5, U5 TLV75533PDBVR

Commit message: Add representative button, axis, hat, encoder and switch examples
Parts:
- removed J5: GPIO 3V3, KiCad:PinHeader_1x06_P2.54mm_Vertical, symbol KiCad:Conn_01x06
Connections:
- net HAT_W: now reaches U1.17 (PA6)
- net ENC_A: now reaches U1.18 (PA7)
- net TOGGLE: now reaches U1.20 (PB1)
- net SELECT_LOW: now reaches U1.21 (PB2)
- net ENC_B: now reaches U1.28 (PA8)
- net ENC_PUSH: now reaches U1.37 (PA15)
- net SELECT_HIGH: now reaches U1.42 (PB3)
- net PA1 renamed AXIS_ADC
- net PA2 renamed HAT_N
- net PA3 renamed HAT_E
- net PA4 renamed HAT_S
- no-connect marks 32 -> 25
Other:
- added sheet Input examples (inputs.kicad_sch)
- note added: "SWD and physical test input"
- note removed: "SWD, GPIO and physical test input"

Commit message: Review compact four-layer PCB and add milling qualification coupon
Parts:
- removed D2, D3: SS14, KiCad:D_SMA, symbol KiCad:D_Schottky
- added C13: 100nF 25V X7R, KiCad:C_0805_2012Metric, symbol KiCad:C
- added D5: SMF15A-E3-08, KiCad:D_SMF, symbol KiCad:SMF15A
- added U6, U7: LM66100DCKR, OpenSimGear:TI_DCK0006A_SC70-6_LM66100, symbol OpenSimGear:LM66100DCK_OR
- C1, C10, C11, C6, C8, C9: MPN (none) -> C0805C104K3RACTU
- C2: footprint KiCad:C_0805_2012Metric -> KiCad:C_1210_3225Metric; MPN (none) -> GRM32ER71H106KA12L
- C3, C4, C7: MPN (none) -> C2012X7R1E105K125AB
- C5: value 1uF 25V X7R -> 2.2uF 25V X7R; MPN (none) -> C2012X7R1E225K125AB
- D1: MPN (none) -> SS14-E3/61T
- D4: footprint KiCad:LED_0805_2012Metric -> OpenSimGear:LED_Kingbright_AP2012SGC_0805; MPN (none) -> AP2012SGC
- F1: value 0.25A hold / 30V -> 0.25A hold / 24V; footprint KiCad:Fuse_1206_3216Metric -> OpenSimGear:Fuse_Littelfuse_1206L025-24YR; MPN (none) -> 1206L025/24YR
- J1: MPN (none) -> USB4105-GF-A
- J2, J3: footprint KiCad:RJ12_Amphenol_54601-x06_Horizontal -> OpenSimGear:RJ12_Amphenol_RJE051660510H_Horizontal; MPN (none) -> RJE051660510H
- J4: footprint KiCad:PinHeader_1x05_P2.54mm_Vertical -> OpenSimGear:PinHeader_Samtec_TSW-105-07-L-S_P2.54mm_Vertical; MPN (none) -> TSW-105-07-L-S
- J6: footprint KiCad:PinHeader_1x03_P2.54mm_Vertical -> OpenSimGear:PinHeader_Samtec_TSW-103-07-L-S_P2.54mm_Vertical; MPN (none) -> TSW-103-07-L-S
- R1, R2: MPN (none) -> RC0805FR-075K1L
- R3, R5, R6, R7: MPN (none) -> RC0805FR-0710KL
- R4: MPN (none) -> RC0805FR-0715KL
- R8: MPN (none) -> RC0805FR-071KL
- SW1, SW2: footprint KiCad:SW_PUSH_6mm_H5mm -> KiCad:SW_PUSH_6mm_H4.3mm; MPN (none) -> B3F-1002-G
- U1: MPN (none) -> STM32G0B1CBT6
- U2: MPN (none) -> USBLC6-2SC6
- U3: MPN (none) -> TCAN3413D
- U4: MPN (none) -> R-78E5.0-0.5
- U5: MPN (none) -> TLV75533PDBVR
Connections:
- net +3V3: now also C13.1
- net BUCK_5V: now also U6.1 (VIN), U7.3 (~{CE})
- net BUCK_IN: now also D5.1 (A1)
- net GND: now also C13.2, D5.2 (A2), U6.2 (GND), U6.5 (ST), U7.2 (GND), U7.5 (ST)
- net SYS_5V: now also U6.6 (VOUT), U7.6 (VOUT)
- net USB_VBUS: now also U6.3 (~{CE}), U7.1 (VIN)
- no-connect marks 25 -> 27
Other:
- note added: "12V local branch + reverse polarity + ideal-diode OR + TVS + 3V3"
- note removed: "12V local branch + reverse polarity + diode OR + 3V3"
